File: 555_module_throu.sch (EAGLE design)
At the start: 11 parts, among them IC2 NE555P

Commit message: added frame
Other:
- note added: "github.com/yoshco/555brain"
- moved on the sheet: C1, C2, D1, IC2, JP1, JP2, JP7, R1, R2, R3, R4
