File: 555_module_throu.brd (EAGLE design)
At the start: 34 x 27.9 mm, 11 parts, among them IC2 NE555P

Commit message: papercut sessions
added files used in generating paper cut
https://www.youtube.com/watch?v=Gg8W51C2M4U
Routing:
- net N$1: track 25.2 -> 31.8 mm
- net VCC: track 90.7 -> 92.6 mm
- net N$2: track 12.9 -> 14.0 mm
- net GND: track 58.6 -> 59.7 mm
Changed lines of the file:
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@@
 <setting verticaltext="up"/>
 </settings>
-<grid distance="0.05" unitdist="inch" unit="inch" style="lines" multiple="1" display="yes" altdistance="0.025" altunitdist="inch" altunit="inch"/>
+<grid distance="0.05" unitdist="inch" unit="inch" style="lines" multiple="1" display="no" altdistance="0.025" altunitdist="inch" altunit="inch"/>
 <layers>
 <layer number="1" name="Top" color="4" fill="1" visible="yes" active="yes"/>
@@
 </element>
 <element name="JP2" library="microbuilder" package="1X02_OVAL" value="4.5-5.5V" x="3.81" y="25.4" smashed="yes" rot="R180">
-<attribute name="NAME" x="6.4262" y="23.5712" size="0.8128" layer="25" ratio="18" rot="R180"/>
+<attribute name="NAME" x="7.6962" y="24.8412" size="0.8128" layer="25" ratio="18" rot="R180"/>
 <attribute name="VALUE" x="2.54" y="23.495" size="0.4064" layer="27" ratio="10" rot="R180"/>
 </element>
@@
 <contactref element="JP1" pad="1"/>
 <contactref element="JP2" pad="1"/>
-<wire x1="3.81" y1="12.7" x2="12.7" y2="15.24" width="1.016" layer="1"/>
+<wire x1="3.81" y1="12.7" x2="7.62" y2="12.7" width="1.016" layer="1"/>
+<wire x1="7.62" y1="12.7" x2="7.62" y2="15.24" width="1.016" layer="1"/>
+<wire x1="7.62" y1="15.24" x2="12.7" y2="15.24" width="1.016" layer="1"/>
 <wire x1="15.24" y1="7.62" x2="25.4" y2="7.62" width="1.016" layer="1"/>
 <wire x1="25.4" y1="7.62" x2="25.4" y2="8.8138" width="1.016" layer="1"/>
-<wire x1="20.32" y1="26.67" x2="33.02" y2="26.67" width="1.016" layer="1"/>
 <wire x1="33.02" y1="26.67" x2="33.02" y2="8.89" width="1.016" layer="1"/>
 <wire x1="33.02" y1="8.89" x2="25.4" y2="8.8138" width="1.016" layer="1"/>
-<wire x1="22.86" y1="24.13" x2="20.32" y2="22.86" width="1.016" layer="1"/>
 <wire x1="20.32" y1="26.67" x2="20.32" y2="25.4" width="1.016" layer="1"/>
-<wire x1="20.32" y1="25.4" x2="20.32" y2="22.86" width="1.016" layer="1"/>
+<wire x1="20.32" y1="25.4" x2="20.32" y2="24.13" width="1.016" layer="1"/>
+<wire x1="20.32" y1="24.13" x2="20.32" y2="22.86" width="1.016" layer="1"/>
 <wire x1="5.08" y1="25.4" x2="20.32" y2="25.4" width="1.016" layer="1"/>
 <wire x1="12.7" y1="15.24" x2="15.24" y2="15.24" width="1.016" layer="1"/>
 <wire x1="15.24" y1="15.24" x2="15.24" y2="7.62" width="1.016" layer="1"/>
+<wire x1="22.86" y1="24.13" x2="20.32" y2="24.13" width="1.016" layer="1"/>
+<wire x1="20.32" y1="26.67" x2="33.02" y2="26.67" width="1.016" layer="1"/>
 </signal>
 <signal name="GND">
@@
 <wire x1="2.54" y1="25.4" x2="2.560078125" y2="22.850159375" width="1.016" layer="1"/>
 <wire x1="2.560078125" y1="22.850159375" x2="2.58" y2="20.32" width="1.016" layer="1"/>
-<wire x1="2.58" y1="20.32" x2="1.27" y2="16.51" width="1.016" layer="1"/>
 <wire x1="1.27" y1="16.51" x2="1.27" y2="7.62" width="1.016" layer="1"/>
 <wire x1="1.27" y1="7.62" x2="3.81" y2="7.62" width="1.016" layer="1"/>
@@
 <wire x1="25.4" y1="2.54" x2="10.16" y2="2.54" width="1.016" layer="1"/>
 <wire x1="10.16" y1="2.54" x2="10.16" y2="7.62" width="1.016" layer="1"/>
+<wire x1="2.58" y1="20.32" x2="2.54" y2="20.32" width="1.016" layer="1"/>
+<wire x1="2.54" y1="20.32" x2="2.54" y2="16.51" width="1.016" layer="1"/>
+<wire x1="2.54" y1="16.51" x2="1.27" y2="16.51" width="1.016" layer="1"/>
 </signal>
 <signal name="N$1">
@@
 <contactref element="IC2" pad="2"/>
 <wire x1="7.58" y1="20.32" x2="12.7" y2="20.32" width="1.016" layer="1"/>
-<wire x1="12.7" y1="20.32" x2="20.32" y2="17.78" width="1.016" layer="1"/>
-<wire x1="20.32" y1="17.78" x2="25.4" y2="13.97" width="1.016" layer="1"/>
-<wire x1="25.4" y1="13.97" x2="30.48" y2="11.43" width="1.016" layer="1"/>
+<wire x1="12.7" y1="20.32" x2="16.51" y2="20.32" width="1.016" layer="1"/>
+<wire x1="16.51" y1="20.32" x2="16.51" y2="17.78" width="1.016" layer="1"/>
+<wire x1="16.51" y1="17.78" x2="20.32" y2="17.78" width="1.016" layer="1"/>
+<wire x1="20.32" y1="17.78" x2="25.4" y2="17.78" width="1.016" layer="1"/>
+<wire x1="25.4" y1="17.78" x2="25.4" y2="13.97" width="1.016" layer="1"/>
+<wire x1="25.4" y1="13.97" x2="30.48" y2="13.97" width="1.016" layer="1"/>
+<wire x1="30.48" y1="13.97" x2="30.48" y2="11.43" width="1.016" layer="1"/>
 </signal>
 <signal name="N$2">
@@
 <contactref element="D1" pad="A"/>
 <contactref element="IC2" pad="7"/>
-<wire x1="20.32" y1="20.32" x2="25.4" y2="21.59" width="1.016" layer="1"/>
+<wire x1="20.32" y1="20.32" x2="22.86" y2="20.32" width="1.016" layer="1"/>
+<wire x1="22.86" y1="20.32" x2="22.86" y2="21.59" width="1.016" layer="1"/>
+<wire x1="22.86" y1="21.59" x2="25.4" y2="21.59" width="1.016" layer="1"/>
 <wire x1="25.4" y1="21.59" x2="30.48" y2="21.59" width="1.016" layer="1"/>
 <wire x1="30.48" y1="24.13" x2="30.48" y2="21.59" width="1.016" layer="1"/>
