File: 555srvc.sch (EAGLE design)
At the start: 10 parts, among them IC1 555

Commit message: board layout
Parts:
- C2: value 1000UF -> (none); device Panasonic-EEE0_EEE1_EEE2_EEEFC:EEE-1AA102P-CASE-G -> adafruit:CPOL-USE5-6
- JP2, JP3: device adafruit:PINHD-1X3 -> adafruit:PINHD-1X3CB
Connections:
- net GND: now also C2.-, JP3.1; no longer C2.2, JP3.2
- net VCC: now also C2.+, JP3.2; no longer C2.1, JP3.1
Changed lines of the file:
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@@
 <grid distance="0.1" unitdist="inch" unit="inch" style="lines" multiple="1" display="no" altdistance="0.01" altunitdist="inch" altunit="inch"/>
 <layers>
-<layer number="1" name="Top" color="4" fill="1" visible="yes" active="no"/>
-<layer number="16" name="Bottom" color="1" fill="1" visible="yes" active="no"/>
-<layer number="17" name="Pads" color="2" fill="1" visible="yes" active="no"/>
-<layer number="18" name="Vias" color="2" fill="1" visible="yes" active="no"/>
-<layer number="19" name="Unrouted" color="6" fill="1" visible="yes" active="no"/>
-<layer number="20" name="Dimension" color="15" fill="1" visible="yes" active="no"/>
-<layer number="21" name="tPlace" color="7" fill="1" visible="yes" active="no"/>
-<layer number="22" name="bPlace" color="7" fill="1" visible="yes" active="no"/>
-<layer number="23" name="tOrigins" color="15" fill="1" visible="yes" active="no"/>
-<layer number="24" name="bOrigins" color="15" fill="1" visible="yes" active="no"/>
-<layer number="25" name="tNames" color="7" fill="1" visible="yes" active="no"/>
-<layer number="26" name="bNames" color="7" fill="1" visible="yes" active="no"/>
-<layer number="27" name="tValues" color="7" fill="1" visible="yes" active="no"/>
-<layer number="28" name="bValues" color="7" fill="1" visible="yes" active="no"/>
+<layer number="1" name="Top" color="4" fill="1" visible="no" active="no"/>
+<layer number="16" name="Bottom" color="1" fill="1" visible="no" active="no"/>
+<layer number="17" name="Pads" color="2" fill="1" visible="no" active="no"/>
+<layer number="18" name="Vias" color="2" fill="1" visible="no" active="no"/>
+<layer number="19" name="Unrouted" color="6" fill="1" visible="no" active="no"/>
+<layer number="20" name="Dimension" color="15" fill="1" visible="no" active="no"/>
+<layer number="21" name="tPlace" color="7" fill="1" visible="no" active="no"/>
+<layer number="22" name="bPlace" color="7" fill="1" visible="no" active="no"/>
+<layer number="23" name="tOrigins" color="15" fill="1" visible="no" active="no"/>
+<layer number="24" name="bOrigins" color="15" fill="1" visible="no" active="no"/>
+<layer number="25" name="tNames" color="7" fill="1" visible="no" active="no"/>
+<layer number="26" name="bNames" color="7" fill="1" visible="no" active="no"/>
+<layer number="27" name="tValues" color="7" fill="1" visible="no" active="no"/>
+<layer number="28" name="bValues" color="7" fill="1" visible="no" active="no"/>
 <layer number="29" name="tStop" color="7" fill="3" visible="no" active="no"/>
 <layer number="30" name="bStop" color="7" fill="6" visible="no" active="no"/>
@@
 <layer number="35" name="tGlue" color="7" fill="4" visible="no" active="no"/>
 <layer number="36" name="bGlue" color="7" fill="5" visible="no" active="no"/>
-<layer number="37" name="tTest" color="7" fill="1" visible="yes" active="no"/>
-<layer number="38" name="bTest" color="7" fill="1" visible="yes" active="no"/>
+<layer number="37" name="tTest" color="7" fill="1" visible="no" active="no"/>
+<layer number="38" name="bTest" color="7" fill="1" visible="no" active="no"/>
 <layer number="39" name="tKeepout" color="4" fill="11" visible="no" active="no"/>
 <layer number="40" name="bKeepout" color="1" fill="11" visible="no" active="no"/>
@@
 <layer number="44" name="Drills" color="7" fill="1" visible="no" active="no"/>
 <layer number="45" name="Holes" color="7" fill="1" visible="no" active="no"/>
-<layer number="46" name="Milling" color="3" fill="1" visible="yes" active="no"/>
-<layer number="47" name="Measures" color="7" fill="1" visible="yes" active="no"/>
-<layer number="48" name="Document" color="7" fill="1" visible="yes" active="no"/>
-<layer number="49" name="Reference" color="7" fill="1" visible="yes" active="no"/>
-<layer number="50" name="dxf" color="7" fill="1" visible="yes" active="no"/>
-<layer number="51" name="tDocu" color="7" fill="1" visible="yes" active="no"/>
-<layer number="52" name="bDocu" color="7" fill="1" visible="yes" active="no"/>
-<layer number="53" name="tGND_GNDA" color="7" fill="9" visible="yes" active="no"/>
-<layer number="54" name="bGND_GNDA" color="1" fill="9" visible="yes" active="no"/>
-<layer number="56" name="wert" color="7" fill="1" visible="yes" active="no"/>
-<layer number="57" name="tCAD" color="7" fill="1" visible="yes" active="no"/>
+<layer number="46" name="Milling" color="3" fill="1" visible="no" active="no"/>
+<layer number="47" name="Measures" color="7" fill="1" visible="no" active="no"/>
+<layer number="48" name="Document" color="7" fill="1" visible="no" active="no"/>
+<layer number="49" name="Reference" color="7" fill="1" visible="no" active="no"/>
+<layer number="50" name="dxf" color="7" fill="1" visible="no" active="no"/>
+<layer number="51" name="tDocu" color="7" fill="1" visible="no" active="no"/>
+<layer number="52" name="bDocu" color="7" fill="1" visible="no" active="no"/>
+<layer number="53" name="tGND_GNDA" color="7" fill="9" visible="no" active="no"/>
+<layer number="54" name="bGND_GNDA" color="1" fill="9" visible="no" active="no"/>
+<layer number="56" name="wert" color="7" fill="1" visible="no" active="no"/>
+<layer number="57" name="tCAD" color="7" fill="1" visible="no" active="no"/>
 <layer number="90" name="Modules" color="5" fill="1" visible="yes" active="yes"/>
 <layer number="91" name="Nets" color="2" fill="1" visible="yes" active="yes"/>
@@
 <part name="P+1" library="microbuilder" deviceset="VCC" device=""/>
 <part name="U$1" library="microbuilder" deviceset="GND" device=""/>
-<part name="C2" library="Panasonic-EEE0_EEE1_EEE2_EEEFC" deviceset="EEE-" device="-CASE-G" technology="1AA102P" value="1000UF"/>
 <part name="P+2" library="microbuilder" deviceset="VCC" device=""/>
 <part name="C1" library="ATtami" deviceset="RESISTOR" device="0805-RES" value="1uF"/>
 <part name="P+5" library="microbuilder" deviceset="VCC" device=""/>
 <part name="U$3" library="microbuilder" deviceset="GND" device=""/>
-<part name="JP2" library="adafruit" deviceset="PINHD-1X3" device="" value="SERVO_OUT"/>
-<part name="JP3" library="adafruit" deviceset="PINHD-1X3" device="" value="INPUT / CV"/>
+<part name="JP2" library="adafruit" deviceset="PINHD-1X3" device="CB" value="SERVO_OUT"/>
+<part name="JP3" library="adafruit" deviceset="PINHD-1X3" device="CB" value="INPUT / CV"/>
 <part name="P+6" library="microbuilder" deviceset="VCC" device=""/>
 <part name="U$4" library="microbuilder" deviceset="GND" device=""/>
 <part name="FRAME1" library="frames" deviceset="A5L-LOC" device=""/>
 <part name="P+3" library="microbuilder" deviceset="VCC" device=""/>
+<part name="C2" library="adafruit" deviceset="CPOL-US" device="E5-6"/>
 </parts>
 <sheets>
@@
 <instance part="P+1" gate="VCC" x="68.58" y="71.12"/>
 <instance part="U$1" gate="G$1" x="53.34" y="38.1"/>
-<instance part="C2" gate="A" x="66.04" y="35.56" smashed="yes" rot="R90">
-<attribute name="NAME" x="65.4304" y="42.6974" size="2.0828" layer="95" ratio="10" rot="SR180"/>
-<attribute name="VALUE" x="66.7258" y="36.0426" size="2.0828" layer="96" ratio="10" rot="SR0"/>
-</instance>
 <instance part="P+2" gate="VCC" x="25.4" y="40.64" rot="R180"/>
 <instance part="C1" gate="G$1" x="45.72" y="43.18" smashed="yes">
@@
 <attribute name="VALUE" x="95.25" y="43.18" size="1.778" layer="96"/>
 </instance>
-<instance part="P+6" gate="VCC" x="86.36" y="55.88" smashed="yes">
-<attribute name="VALUE" x="82.042" y="52.832" size="1.27" layer="96"/>
-</instance>
-<instance part="U$4" gate="G$1" x="86.36" y="48.26"/>
+<instance part="P+6" gate="VCC" x="86.36" y="53.34" smashed="yes">
+<attribute name="VALUE" x="84.074" y="49.022" size="1.27" layer="96"/>
+</instance>
+<instance part="U$4" gate="G$1" x="91.44" y="53.34" rot="R270"/>
 <instance part="FRAME1" gate="G$1" x="0" y="0"/>
 <instance part="P+3" gate="VCC" x="66.04" y="30.48" rot="R180"/>
+<instance part="C2" gate="G$1" x="66.04" y="38.1" rot="R180"/>
 </instances>
 <busses>
@@
 </segment>
 <segment>
-<pinref part="P+6" gate="VCC" pin="VCC"/>
-<pinref part="JP3" gate="A" pin="1"/>
-<wire x1="86.36" y1="53.34" x2="99.06" y2="53.34" width="0.1524" layer="91"/>
-</segment>
-<segment>
-<pinref part="C2" gate="A" pin="1"/>
 <pinref part="P+3" gate="VCC" pin="VCC"/>
 <wire x1="66.04" y1="33.02" x2="66.04" y2="35.56" width="0.1524" layer="91"/>
+<pinref part="C2" gate="G$1" pin="+"/>
+</segment>
+<segment>
+<pinref part="JP3" gate="A" pin="2"/>
+<pinref part="P+6" gate="VCC" pin="VCC"/>
+<wire x1="99.06" y1="50.8" x2="86.36" y2="50.8" width="0.1524" layer="91"/>
 </segment>
 </net>
@@
 <pinref part="JP2" gate="A" pin="2"/>
 <wire x1="86.36" y1="66.04" x2="99.06" y2="66.04" width="0.1524" layer="91"/>
-</segment>
-<segment>
-<pinref part="U$4" gate="G$1" pin="GND"/>
-<pinref part="JP3" gate="A" pin="2"/>
-<wire x1="86.36" y1="50.8" x2="99.06" y2="50.8" width="0.1524" layer="91"/>
 </segment>
 <segment>
@@
 <wire x1="50.8" y1="43.18" x2="53.34" y2="43.18" width="0.1524" layer="91"/>
 <junction x="53.34" y="43.18"/>
-<pinref part="C2" gate="A" pin="2"/>
+<pinref part="C2" gate="G$1" pin="-"/>
 <junction x="66.04" y="43.18"/>
 </segment>
+<segment>
+<pinref part="U$4" gate="G$1" pin="GND"/>
+<pinref part="JP3" gate="A" pin="1"/>
+<wire x1="93.98" y1="53.34" x2="99.06" y2="53.34" width="0.1524" layer="91"/>
+</segment>
 </net>
